Commit message: Required folders

File: arena_with_qr/models/diff_drive/diff_drive.xacro (robot description, xacro)
@@ -2,5 +2,4 @@
 <!-- choose a name space and start xacro -->
 <robot name="ddrbot" xmlns:xacro="http://wwww.ros.org/wiki/xacro">
-    <pose>-1.201849 -1.539665 0.170097 0 0 1.595502</pose>
  <!-- Start by including all the required xacro files which hold the macros -->
  <xacro:include filename="$(find arena_with_qr)/models/diff_drive/diff_drive.gazebo" />
@@ -10,5 +9,4 @@
  <!-- Create a dummy link as a base link -->
   <link name='base_link'>
-    <pose>-1.201849 -1.539665 0.170097 0 0 1.595502</pose>
   </link>
   <joint type="fixed" name="base_link_to_chassis">
@@ -62,12 +60,12 @@
     </visual>
     <inertial>
-      <!-- <origin xyz="0 0 0" rpy="0 1.5707 1.5707"/> -->
+      <origin xyz="${-(r_wheel/2)+x_chassis/2} 0 ${-z_chassis+cr_wheel}" rpy="0 0 0"/>
       <mass value="${cm_wheel}"/>
-      <castor_inertia m="${cm_wheel}" r="${cr_wheel}" />
-      <!-- <xacro:castor_inertia m="${cm_wheel}" r="${cr_wheel}" /> -->
+      <!-- <castor_inertia m="${cm_wheel}" r="${cr_wheel}" /> -->
+      <xacro:castor_inertia m="${cm_wheel}" r="${cr_wheel}" />
     </inertial>
    <!-- Adding the left clamp -->
    <collision name='left_clamp_collision'>
-      <origin xyz="${(x_left_clamp/2)+x_chassis/2} ${y_chassis/2-y_left_clamp/2} 0" rpy="0 0 0"/>
+      <origin xyz="${(x_left_clamp/2)+x_chassis/2} ${y_chassis/2+x_left_clamp/2-y_left_clamp/2} 0" rpy="0 0 0"/>
       <geometry>
        <box size="${x_left_clamp} ${y_left_clamp} ${z_left_clamp}"/>
@@ -85,5 +83,5 @@
     </collision>
     <visual name='left_clamp_visual'>
-	    <origin xyz="${(x_left_clamp/2)+x_chassis/2} ${y_chassis/2-y_left_clamp/2} 0" rpy="0 0 0"/>
+	    <origin xyz="${(x_left_clamp/2)+x_chassis/2} ${y_chassis/2+x_left_clamp/2-y_left_clamp/2} 0" rpy="0 0 0"/>
     	<geometry>
         <box size="${x_left_clamp} ${y_left_clamp} ${z_left_clamp}"/>
@@ -95,6 +93,6 @@
     </inertial>
    <!-- Adding the right clamp -->
-   <collision name='right clamp_collision'>
-      <origin xyz="${(x_right_clamp/2)+x_chassis/2} ${-(y_chassis/2)+y_right_clamp/2} 0" rpy="0 0 0"/>
+   <collision name='right_clamp_collision'>
+      <origin xyz="${(x_left_clamp/2)+x_chassis/2} ${-(y_chassis/2)-x_right_clamp/2+y_left_clamp/2} 0" rpy="0 0 0"/>
       <geometry>
        <box size="${x_right_clamp} ${y_right_clamp} ${z_right_clamp}"/>
@@ -111,8 +109,62 @@
       </surface>
     </collision>
-    <visual name='caster_visual'>
-	    <origin xyz="${(x_right_clamp/2)+x_chassis/2} ${-(y_chassis/2)+y_right_clamp/2} 0" rpy="0 0 0"/>
+    <visual name='right_clamp_visual'>
+	    <origin xyz="${(x_left_clamp/2)+x_chassis/2} ${-(y_chassis/2)-x_right_clamp/2+y_left_clamp/2} 0" rpy="0 0 0"/>
     	<geometry>
         <box size="${x_right_clamp} ${y_right_clamp} ${z_right_clamp}"/>
+      </geometry>
+    </visual>
+    <inertial>
+      <mass value="${m_right_clamp}"/>
+      <xacro:box_inertia m="${m_right_clamp}" x="${x_right_clamp}" y="${y_right_clamp}" z="${z_right_clamp}"/>
+    </inertial>
+   <!-- Adding the bottom left clamp -->
+   <collision name='bot_left_clamp_collision'>
+      <origin xyz="${x_chassis/2-y_left_clamp/2} ${y_chassis/2+x_left_clamp/4} 0" rpy="0 0 1.570896"/>
+      <geometry>
+       <box size="${x_left_clamp/2} ${y_left_clamp} ${z_left_clamp}"/>
+      </geometry>
+      <surface>
+       <friction>
+        <ode>
+         <mu>0</mu>
+         <mu2>0</mu2>
+         <slip1>0</slip1>
+         <slip2>0</slip2>
+        </ode>
+       </friction>
+      </surface>
+    </collision>
+    <visual name='bot_left_clamp_visual'>
+	    <origin xyz="${x_chassis/2-y_left_clamp/2} ${y_chassis/2+x_left_clamp/4} 0" rpy="0 0 1.570896"/>
+    	<geometry>
+        <box size="${x_left_clamp/2} ${y_left_clamp} ${z_left_clamp}"/>
+      </geometry>
+    </visual>
+    <inertial>
+      <mass value="${m_left_clamp}"/>
+      <xacro:box_inertia m="${m_left_clamp}" x="${x_left_clamp}" y="${y_left_clamp}" z="${z_left_clamp}"/>
+    </inertial>
+   <!-- Adding the bottom right clamp -->
+   <collision name='bot_right_clamp_collision'>
+      <origin xyz="${x_chassis/2-y_right_clamp/2} ${-(y_chassis/2)-x_right_clamp/4} 0" rpy="0 0 -1.570896"/>
+      <geometry>
+       <box size="${x_right_clamp/2} ${y_right_clamp} ${z_right_clamp}"/>
+      </geometry>
+      <surface>
+       <friction>
+        <ode>
+         <mu>0</mu>
+         <mu2>0</mu2>
+         <slip1>0</slip1>
+         <slip2>0</slip2>
+        </ode>
+       </friction>
+      </surface>
+    </collision>
+    <visual name='bot_right_clamp_visual'>
+	    <origin xyz="${x_chassis/2-y_right_clamp/2} ${-(y_chassis/2)-x_right_clamp/4} 0" rpy="0 0 -1.570896"/>
+    	<geometry>
+        <box size="${x_right_clamp/2} ${y_right_clamp} ${z_right_clamp}"/>
       </geometry>
     </visual>
@@ -149,6 +201,6 @@
       <origin xyz="0 0 0" rpy="0 1.5707 1.5707"/>
       <mass value="${m_wheel}"/>
-      <cylinder_inertia m="${m_wheel}" r="${r_wheel}" h="${h_wheel}"/>
-      <!-- <xacro:cylinder_inertia m="${m_wheel}" r="${r_wheel}" h="${h_wheel}"/> -->
+      <!-- <cylinder_inertia m="${m_wheel}" r="${r_wheel}" h="${h_wheel}"/> -->
+      <xacro:cylinder_inertia m="${m_wheel}" r="${r_wheel}" h="${h_wheel}"/>
     </inertial>
   </link>
@@ -179,6 +231,6 @@
       <origin xyz="0 0 0" rpy="0 1.5707 1.5707"/>
       <mass value="${m_wheel}"/>
-      <cylinder_inertia m="${m_wheel}" r="${r_wheel}" h="${h_wheel}"/>
-      <!-- <xacro:cylinder_inertia m="${m_wheel}" r="${r_wheel}" h="${h_wheel}"/> -->
+      <!-- <cylinder_inertia m="${m_wheel}" r="${r_wheel}" h="${h_wheel}"/> -->
+      <xacro:cylinder_inertia m="${m_wheel}" r="${r_wheel}" h="${h_wheel}"/>
     </inertial>
   </link>
@@ -206,10 +258,4 @@
     <child link="camera_link1"/>
   </joint>
-  <joint name="camera_joint2" type="fixed">
-    <axis xyz="0 0 1" />
-    <origin xyz="${x_chassis/8} 0 ${-z_chassis+2*cr_wheel}" rpy="0 1.570896 0"/>
-    <parent link="base_link"/>
-    <child link="camera_link2"/>
-  </joint>
   <joint name="laser_joint1" type="fixed">
     <axis xyz="1 0 0" />
@@ -218,28 +264,4 @@
     <child link="laser_link1"/>
   </joint>
-  <joint name="laser_joint2" type="fixed">
-    <axis xyz="0 0 1" />
-    <origin xyz="${x_chassis/4} ${y_chassis/4} ${-z_chassis+2*cr_wheel}" rpy="0 1.570896 0"/>
-    <parent link="base_link"/>
-    <child link="laser_link2"/>
-  </joint>
-  <joint name="laser_joint3" type="fixed">
-    <axis xyz="0 0 1" />
-    <origin xyz="${x_chassis/4} ${y_chassis/8} ${-z_chassis+2*cr_wheel}" rpy="0 1.570896 0"/>
-    <parent link="base_link"/>
-    <child link="laser_link3"/>
-  </joint>
-  <joint name="laser_joint4" type="fixed">
-    <axis xyz="0 0 1" />
-    <origin xyz="${x_chassis/4} ${-y_chassis/8} ${-z_chassis+2*cr_wheel}" rpy="0 1.570896 0"/>
-    <parent link="base_link"/>
-    <child link="laser_link4"/>
-  </joint>
-  <joint name="laser_joint5" type="fixed">
-    <axis xyz="0 0 1" />
-    <origin xyz="${x_chassis/4} ${-y_chassis/4} ${-z_chassis+2*cr_wheel}" rpy="0 1.570896 0"/>
-    <parent link="base_link"/>
-    <child link="laser_link5"/>
-  </joint>
   <joint name="laser_joint6" type="fixed">
     <axis xyz="1 0 0" />
@@ -264,25 +286,5 @@
     </visual>
     <inertial>
-      <mass value="0.15" />
-      <origin xyz="0 0 0" rpy="0 0 0"/>
-      <inertia ixx="1e-6" ixy="0" ixz="0" iyy="1e-6" iyz="0" izz="1e-6" />
-    </inertial>
-  </link>
-  <link name="camera_link2">
-    <collision>
-      <origin xyz="0 0 0" rpy="0 0 0"/>
-      <geometry>
-    <box size="${camera_link} ${camera_link} ${camera_link}"/>
-      </geometry>
-    </collision>
-    <visual>
-      <origin xyz="0 0 0" rpy="0 0 0"/>
-      <geometry>
-    <box size="${camera_link} ${camera_link} ${camera_link}"/>
-      </geometry>
-      <material name="red"/>
-    </visual>
-    <inertial>
-      <mass value="0.1" />
+      <mass value="0.2" />
       <origin xyz="0 0 0" rpy="0 0 0"/>
       <inertia ixx="1e-6" ixy="0" ixz="0" iyy="1e-6" iyz="0" izz="1e-6" />
@@ -305,85 +307,5 @@
     </visual>
     <inertial>
-      <mass value="0.05" />
-      <origin xyz="0 0 0" rpy="0 0 0"/>
-      <inertia ixx="1e-6" ixy="0" ixz="0" iyy="1e-6" iyz="0" izz="1e-6" />
-    </inertial>
-  </link>
-  <link name="laser_link2">
-    <collision>
-      <origin xyz="0 0 0" rpy="0 0 0"/>
-      <geometry>
-    <box size="${laser_link} ${laser_link} ${laser_link}"/>
-      </geometry>
-    </collision>
-    <visual>
-      <origin xyz="0 0 0" rpy="0 0 0"/>
-      <geometry>
-    <box size="${laser_link} ${laser_link} ${laser_link}"/>
-      </geometry>
-      <material name="red"/>
-    </visual>
-    <inertial>
-      <mass value="0.01" />
-      <origin xyz="0 0 0" rpy="0 0 0"/>
-      <inertia ixx="1e-6" ixy="0" ixz="0" iyy="1e-6" iyz="0" izz="1e-6" />
-    </inertial>
-  </link>
-  <link name="laser_link3">
-    <collision>
-      <origin xyz="0 0 0" rpy="0 0 0"/>
-      <geometry>
-    <box size="${laser_link} ${laser_link} ${laser_link}"/>
-      </geometry>
-    </collision>
-    <visual>
-      <origin xyz="0 0 0" rpy="0 0 0"/>
-      <geometry>
-    <box size="${laser_link} ${laser_link} ${laser_link}"/>
-      </geometry>
-      <material name="red"/>
-    </visual>
-    <inertial>
-      <mass value="0.01" />
-      <origin xyz="0 0 0" rpy="0 0 0"/>
-      <inertia ixx="1e-6" ixy="0" ixz="0" iyy="1e-6" iyz="0" izz="1e-6" />
-    </inertial>
-  </link>
-  <link name="laser_link4">
-    <collision>
-      <origin xyz="0 0 0" rpy="0 0 0"/>
-      <geometry>
-    <box size="${laser_link} ${laser_link} ${laser_link}"/>
-      </geometry>
-    </collision>
-    <visual>
-      <origin xyz="0 0 0" rpy="0 0 0"/>
-      <geometry>
-    <box size="${laser_link} ${laser_link} ${laser_link}"/>
-      </geometry>
-      <material name="red"/>
-    </visual>
-    <inertial>
-      <mass value="0.01" />
-      <origin xyz="0 0 0" rpy="0 0 0"/>
-      <inertia ixx="1e-6" ixy="0" ixz="0" iyy="1e-6" iyz="0" izz="1e-6" />
-    </inertial>
-  </link>
-  <link name="laser_link5">
-    <collision>
-      <origin xyz="0 0 0" rpy="0 0 0"/>
-      <geometry>
-    <box size="${laser_link} ${laser_link} ${laser_link}"/>
-      </geometry>
-    </collision>
-    <visual>
-      <origin xyz="0 0 0" rpy="0 0 0"/>
-      <geometry>
-    <box size="${laser_link} ${laser_link} ${laser_link}"/>
-      </geometry>
-      <material name="red"/>
-    </visual>
-    <inertial>
-      <mass value="0.01" />
+      <mass value="0.15" />
       <origin xyz="0 0 0" rpy="0 0 0"/>
       <inertia ixx="1e-6" ixy="0" ixz="0" iyy="1e-6" iyz="0" izz="1e-6" />
@@ -405,5 +327,5 @@
     </visual>
     <inertial>
-      <mass value="0.05" />
+      <mass value="0.15" />
       <origin xyz="0 0 0" rpy="0 0 0"/>
       <inertia ixx="1e-6" ixy="0" ixz="0" iyy="1e-6" iyz="0" izz="1e-6" />

File: arena_with_qr/models/diff_drive/parameter.xacro (robot description, xacro)
@@ -6,5 +6,5 @@
  <xacro:property name="y_chassis" value="0.12" />
  <xacro:property name="z_chassis" value="0.05" />
- <xacro:property name="m_chassis" value="0.6" />
+ <xacro:property name="m_chassis" value="0.7" />
  <!-- Parameter for the chassis, size [m] and mass [kg] -->
  <xacro:property name="x_left_clamp" value="0.04" />
